File: Draft 2.brd (EAGLE design)
At the start: 127 x 127 mm, 41 parts, among them IC1 74HC04D-Q100,118, IC2 CNY17F-3X007, IC3 CNY17F-3X007, J1 N2534-6V0C-RB-WF, J10 691305540002, J11 CON-SOCJ-2155, J12 TB002-500-03BE, J13 TB002-500-03BE, J14 TB002-500-03BE, J2 73131-0240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

Commit message: auto push run at Mon 24 Aug 2020 01:14:17 AM EDT
Parts:
- moved TP1 139.4 mm to (-6.35, -3.81)
Connections:
- net N$10 renamed 3A
- net N$11 renamed COAX4
- net N$12 renamed COAX5
- net N$13 renamed COAX6
- net N$14 renamed TERM1
- net N$17 renamed TERM2
- net N$18 renamed TERM3
- net N$2 renamed C
- net N$25 renamed 1Y
- net N$26 renamed 2A
- net N$27 renamed 3Y
- net N$28 renamed 4A
- net N$29 renamed 2Y
- net N$30 renamed 4Y
- net N$31 renamed 5Y
- net N$32 renamed JACK13
- net N$33 renamed JACK12
- net N$34 renamed JACK11
- net N$35 renamed JACK10
- net N$36 renamed JACK9
- net N$37 renamed JACK8
- net N$38 renamed JACK7
- net N$39 renamed JACK6
- net N$40 renamed JACK1
- net N$41 renamed JACK2
- net N$42 renamed JACK3
- net N$43 renamed JACK4
- net N$44 renamed 6A
- net N$45 renamed 6Y
- net N$49 renamed JACK5
- net N$6 renamed VCC
- net N$8 renamed 1A
- net N$9 renamed 5A
Routing:
- net JACK13: track 8.89 -> 0.00 mm
- net JACK1: track 7.62 -> 11.0 mm
- net 3A: track 27.9 -> 25.3 mm

Commit message: auto push run at Mon 24 Aug 2020 11:25:32 AM EDT
Parts:
- moved TP1 139.4 mm to (97.8, 88.9)
- moved R1 24.7 mm to (88.9, 119.4)
- moved R2 24.2 mm to (88.9, 108.0)
- moved BR1 23.9 mm to (88.9, 124.5)
- moved R10 20.7 mm to (67.3, 113.0)
- moved IC2 14.5 mm to (76.2, 121.9)
- moved IC3 14.5 mm to (76.2, 110.5)
- moved R9 14.5 mm to (67.3, 124.5)
- moved BR2 10.2 mm to (88.9, 113.0)
- moved C1 4.02 mm to (72.4, 97.8)
- moved IC1 3.59 mm to (68.6, 87.6)
- moved R5 3.59 mm to (114.3, 121.9), turned to 270 degrees
- moved R6 3.59 mm to (114.3, 105.4), turned to 270 degrees
Routing:
- net VCC: track 137.8 -> 0.08 mm, vias 5 -> 0
- net N$6: track 39.9 -> 6.40 mm, vias 3 -> 0
- net N$4: track 33.9 -> 2.59 mm, vias 2 -> 0
- net 4Y: track 132.0 -> 103.5 mm
- net N$16: track 33.2 -> 4.81 mm, vias 3 -> 0
- net 3Y: track 140.9 -> 112.7 mm
- net 5Y: track 94.2 -> 71.1 mm, vias 6 -> 2
- net 6Y: track 89.2 -> 66.9 mm, vias 4 -> 2
- net N$5: track 25.8 -> 6.40 mm
- net 2Y: track 52.6 -> 33.7 mm
- net TERM3: track 51.7 -> 70.3 mm, vias 1 -> 2
- net COAX6: track 141.4 -> 124.3 mm
- net C: track 159.5 -> 175.6 mm
- net 2A: track 34.1 -> 21.8 mm
- net 1Y: track 29.1 -> 41.1 mm
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- added copper zone on layer 16, net GND
- added copper zone on layer 1, net VCC
Other:
- board text added: "Chen-Lab PCB"
- board text added: "RevA (8/2020)"
- board text added: "kremer@bu.edu, edf.bu.edu"
