File: eagle_files/Draft 2.brd (EAGLE design)
At the start: 127 x 127 mm, 41 parts, among them IC1 74HC04D-Q100,118, IC2 CNY17F-3X007, IC3 CNY17F-3X007, J1 N2534-6V0C-RB-WF, J10 691305540002, J11 CON-SOCJ-2155, J12 TB002-500-03BE, J13 TB002-500-03BE, J14 TB002-500-03BE, J2 73131-0240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

Commit message: auto push run at Mon 24 Aug 2020 03:10:38 PM EDT
Parts:
- moved BR2 8.26 mm to (95.5, 108.1), turned to 270 degrees
- moved BR1 8.13 mm to (95.2, 119.4), turned to 270 degrees
- moved Q1 3.81 mm to (102.9, 121.9)
- moved Q2 3.81 mm to (102.9, 110.5)
Connections:
- removed net C: IC2.5, IC3.5, J11.1, Q1.2, Q1.4, Q2.2, Q2.4
- removed net N$15: J9.1, Q1.3, R1.2, R5.2
- removed net N$16: BR1.2, Q1.1
- new net N$11: Q2.1, R2.2, R6.2
- new net N$3: Q1.1, R1.2, R5.2
- new net N$8: BR1.1, BR2.1, IC2.5, IC3.5, J11.1, Q1.2, Q1.4, Q2.2, Q2.4
- net GND: no longer BR1.1, BR2.1
- net N$2: now also J10.1, Q2.3; no longer Q2.1
- net N$7: now also BR1.2, J9.1, Q1.3; no longer J10.1, Q2.3, R2.2, R6.2
Routing:
- net N$8: track 0.00 -> 178.3 mm, vias 0 -> 3
- net C: track 175.6 -> 0.00 mm, vias 3 -> 0
- net N$11: track 0.00 -> 40.7 mm, vias 0 -> 2
- net N$15: track 35.7 -> 0.00 mm
- net N$3: track 0.00 -> 31.3 mm, vias 0 -> 2
- net N$2: track 4.81 -> 32.1 mm
- net GND: track 69.5 -> 63.4 mm, vias 15 -> 13
- net N$16: track 4.81 -> 0.00 mm
- net N$7: track 36.5 -> 32.4 mm
