File: eagle_files/Draft 2.sch (EAGLE design)
At the start: 41 parts, among them IC1 74HC04D-Q100,118, IC2 CNY17F-3X007, IC3 CNY17F-3X007, J1 N2534-6V0C-RB-WF, J10 691305540002, J11 CON-SOCJ-2155, J12 TB002-500-03BE, J13 TB002-500-03BE, J14 TB002-500-03BE, J2 73131-0240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

Commit message: auto push run at Mon 24 Aug 2020 03:10:38 PM EDT
Connections:
- removed net C: IC2.C, IC3.C, J11.1, Q1.C, Q1.C_(TAB), Q2.C, Q2.C_(TAB)
- removed net N$15: J9.1, Q1.E, R1.2, R5.2
- removed net N$16: BR1.A, Q1.B
- new net N$11: Q2.B, R2.2, R6.2
- new net N$3: Q1.B, R1.2, R5.2
- new net N$8: BR1.K, BR2.K, IC2.C, IC3.C, J11.1, Q1.C, Q1.C_(TAB), Q2.C, Q2.C_(TAB)
- net GND: no longer BR1.K, BR2.K
- net N$2: now also J10.1, Q2.E; no longer Q2.B
- net N$7: now also BR1.A, J9.1, Q1.E; no longer J10.1, Q2.E, R2.2, R6.2
Other:
- moved on the sheet: BR1, BR2, IC3, J10, J11, J9, Q1, Q2, R10, R2, R6
