File: board-design/cage-board.kicad_pcb (KiCad board)
At the start: 2 copper layers, 127 x 152.4 mm, 34 parts, among them J1 Jack-DC, J10 73131-0240, J11 73131-0240, J12 73131-0240, J13 Conn_01x02, J14 Conn_01x02, J15 Conn_02x13_test_points, J2 Conn_02x17_Ribbon, J3 TB002-500-03BE, J4 73131-0240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

Commit message: working on resizing board
Parts:
- moved J12 20.3 mm to (83.6, 147.3)
- moved J10 12.7 mm to (83.6, 12.7)
- moved J8 9.27 mm to (83.6, 41.5)
- moved J4 5.84 mm to (83.6, 70.4)
- moved J6 2.41 mm to (83.6, 99.2)
Other:
- board size 127 x 152.4 mm -> 160 x 160 mm
Changed lines of the file:
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@@
-(kicad_pcb (version 20171130) (host pcbnew 5.1.6)
+(kicad_pcb (version 20171130) (host pcbnew 5.1.5+dfsg1-2build2)
   (general
     (thickness 1.6)
@@
   )
   (module chen-lab:BNC-Chen (layer F.Cu)
-    (at 83.566 76.2)
+    (at 83.566 70.358)
     (fp_text reference J4 (at -4.572 -7.874) (layer F.SilkS)
       (effects (font (size 1 1) (thickness 0.15)))
@@
   )
   (module chen-lab:BNC-Chen (layer F.Cu)
-    (at 83.566 101.6)
+    (at 83.566 99.187)
     (fp_text reference J6 (at -4.572 -7.874) (layer F.SilkS)
       (effects (font (size 1 1) (thickness 0.15)))
@@
   )
   (module chen-lab:BNC-Chen (layer F.Cu)
-    (at 83.566 50.8)
+    (at 83.566 41.529)
     (fp_text reference J8 (at -4.572 -7.874) (layer F.SilkS)
       (effects (font (size 1 1) (thickness 0.15)))
@@
   )
   (module chen-lab:BNC-Chen (layer F.Cu)
-    (at 83.566 25.4)
+    (at 83.566 12.7)
     (fp_text reference J10 (at -4.572 -7.874) (layer F.SilkS)
       (effects (font (size 1 1) (thickness 0.15)))
@@
   )
   (module chen-lab:BNC-Chen (layer F.Cu)
-    (at 83.566 127)
+    (at 83.566 147.32)
     (fp_text reference J12 (at -4.572 -7.874) (layer F.SilkS)
       (effects (font (size 1 1) (thickness 0.15)))
@@
     (effects (font (size 1.27 1.27) (thickness 0.1778)) (justify left))
   )
-  (gr_line (start 76.2 0) (end 76.2 152.4) (layer Edge.Cuts) (width 0.127))
-  (gr_line (start 203.2 0) (end 203.2 152.4) (layer Edge.Cuts) (width 0.127))
-  (gr_line (start 76.2 0) (end 203.2 0) (layer Edge.Cuts) (width 0.127))
-  (gr_line (start 76.2 152.4) (end 203.2 152.4) (layer Edge.Cuts) (width 0.127))
+  (gr_line (start 43.18 0) (end 43.18 160.02) (layer Edge.Cuts) (width 0.127))
+  (gr_line (start 203.2 0) (end 203.2 160.02) (layer Edge.Cuts) (width 0.127))
+  (gr_line (start 43.18 0) (end 203.2 0) (layer Edge.Cuts) (width 0.127))
+  (gr_line (start 43.18 160.02) (end 203.2 160.02) (layer Edge.Cuts) (width 0.127))
   (segment (start 183.42 74.2) (end 183.42 71.628) (width 0.25) (layer F.Cu) (net 1))
   (segment (start 185.42 76.2) (end 183.42 74.2) (width 0.25) (layer F.Cu) (net 1))
@@
   (via (at 152.4 102.87) (size 0.8) (drill 0.4) (layers F.Cu B.Cu) (net 30))
   (segment (start 143.067 99.06) (end 142.24 99.06) (width 0.25) (layer F.Cu) (net 31))
-  (segment (start 83.566 127) (end 91.44 127) (width 0.25) (layer F.Cu) (net 31))
   (segment (start 142.24 99.06) (end 120.015 99.06) (width 0.25) (layer F.Cu) (net 31))
-  (segment (start 91.44 107.95) (end 91.44 104.14) (width 0.25) (layer B.Cu) (net 31))
-  (segment (start 91.44 127) (end 91.44 107.95) (width 0.25) (layer B.Cu) (net 31))
-  (via (at 91.44 127) (size 0.8) (drill 0.4) (layers F.Cu B.Cu) (net 31))
   (via (at 91.44 100.584) (size 0.8) (drill 0.4) (layers F.Cu B.Cu) (net 31))
   (segment (start 92.964 99.06) (end 91.44 100.584) (width 0.25) (layer F.Cu) (net 31))
   (segment (start 93.472 99.06) (end 92.964 99.06) (width 0.25) (layer F.Cu) (net 31))
   (segment (start 120.142 99.06) (end 93.472 99.06) (width 0.25) (layer F.Cu) (net 31))
+  (segment (start 83.566 127) (end 91.44 127) (width 0.25) (layer F.Cu) (net 31))
+  (via (at 91.44 127) (size 0.8) (drill 0.4) (layers F.Cu B.Cu) (net 31))
+  (segment (start 91.44 127) (end 91.44 107.95) (width 0.25) (layer B.Cu) (net 31))
+  (segment (start 91.44 107.95) (end 91.44 104.14) (width 0.25) (layer B.Cu) (net 31))
   (segment (start 91.44 100.584) (end 91.44 104.14) (width 0.25) (layer B.Cu) (net 31))
   (segment (start 170.198 97.79) (end 173.482 97.79) (width 0.25) (layer F.Cu) (net 32))
@@
     (polygon
       (pts
-        (xy 202.946 68.072) (xy 167.132 68.072) (xy 167.132 152.146) (xy 76.454 152.146) (xy 76.454 0.254)
+        (xy 202.946 68.072) (xy 167.132 68.072) (xy 167.132 159.385) (xy 43.815 159.385) (xy 43.815 0.254)
         (xy 202.946 0.254)
       )
@@
     (polygon
       (pts
-        (xy 202.946 152.146) (xy 76.454 152.146) (xy 76.454 0.254) (xy 202.946 0.254)
+        (xy 202.565 159.385) (xy 43.815 159.385) (xy 43.815 0.254) (xy 202.946 0.254)
       )
     )
@@
     (polygon
       (pts
-        (xy 202.946 152.146) (xy 169.672 152.146) (xy 169.672 69.85) (xy 202.946 69.85)
+        (xy 202.565 159.385) (xy 169.545 159.385) (xy 169.545 69.85) (xy 202.946 69.85)
       )
     )

Commit message: working on fixing connectors
Parts:
- moved J6 35.9 mm to (50.8, 113.8)
- moved J4 34.2 mm to (50.8, 80.0)
- moved Je 33.0 mm to (50.8, 45.7)
- moved J10 32.8 mm to (50.8, 12.7)
- moved J12 32.8 mm to (50.8, 147.3)
- moved J5 12.7 mm to (195.8, 12.7)
- moved J11 5.08 mm to (195.8, 45.7)
- renumbered J8 to Je
Routing:
- net Net-(J12-Pad1): track 86.7 -> 138.1 mm, vias 2 -> 1
- net Net-(J6-Pad1): track 62.0 -> 110.3 mm, vias 0 -> 1
- net /P0.7: track 107.5 -> 146.2 mm, vias 2 -> 1
- net /P0.6: track 85.2 -> 117.9 mm, vias 2 -> 1
- net /P0.5: track 63.1 -> 92.0 mm
- net Net-(J11-Pad1): track 99.9 -> 104.8 mm
Changed lines of the file:
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@@
     (thickness 1.6)
     (drawings 26)
-    (tracks 273)
+    (tracks 272)
     (zones 0)
     (modules 34)
@@
   )
   (module chen-lab:BNC-Chen (layer F.Cu)
-    (at 83.566 70.358)
+    (at 50.8 80.01)
     (fp_text reference J4 (at -4.572 -7.874) (layer F.SilkS)
       (effects (font (size 1 1) (thickness 0.15)))
@@
   )
   (module chen-lab:BNC-Chen (layer F.Cu)
-    (at 195.834 25.4 180)
+    (at 195.834 12.7 180)
     (fp_text reference J5 (at 5.842 7.874) (layer F.SilkS)
       (effects (font (size 1 1) (thickness 0.15)))
@@
   )
   (module chen-lab:BNC-Chen (layer F.Cu)
-    (at 83.566 99.187)
+    (at 50.8 113.792)
     (fp_text reference J6 (at -4.572 -7.874) (layer F.SilkS)
       (effects (font (size 1 1) (thickness 0.15)))
@@
   )
   (module chen-lab:BNC-Chen (layer F.Cu)
-    (at 83.566 41.529)
-    (fp_text reference J8 (at -4.572 -7.874) (layer F.SilkS)
+    (at 50.8 45.72)
+    (fp_text reference Je (at -4.572 -7.874) (layer F.SilkS)
       (effects (font (size 1 1) (thickness 0.15)))
     )
@@
   )
   (module chen-lab:BNC-Chen (layer F.Cu)
-    (at 83.566 12.7)
+    (at 50.8 12.7)
     (fp_text reference J10 (at -4.572 -7.874) (layer F.SilkS)
       (effects (font (size 1 1) (thickness 0.15)))
@@
   )
   (module chen-lab:BNC-Chen (layer F.Cu)
-    (at 195.834 50.8 180)
+    (at 195.834 45.72 180)
     (fp_text reference J11 (at 5.588 7.747) (layer F.SilkS)
       (effects (font (size 1 1) (thickness 0.15)))
@@
   )
   (module chen-lab:BNC-Chen (layer F.Cu)
-    (at 83.566 147.32)
+    (at 50.8 147.32)
     (fp_text reference J12 (at -4.572 -7.874) (layer F.SilkS)
       (effects (font (size 1 1) (thickness 0.15)))
@@
     (effects (font (size 1.5 1.5) (thickness 0.3)))
   )
-  (gr_text "[Front Edge]" (at 63.2079 83.7057) (layer Cmts.User)
+  (gr_text "[Front Edge]" (at 35.56 83.185) (layer Cmts.User)
     (effects (font (size 1.5 1.5) (thickness 0.3)))
   )
@@
   (segment (start 143.067 95.25) (end 129.525 95.25) (width 0.25) (layer F.Cu) (net 21))
   (segment (start 129.525 95.25) (end 128.524 95.25) (width 0.25) (layer F.Cu) (net 21))
-  (segment (start 83.82 76.454) (end 83.566 76.2) (width 0.25) (layer B.Cu) (net 22))
-  (segment (start 83.82 83.82) (end 83.82 83.566) (width 0.25) (layer B.Cu) (net 22))
-  (segment (start 83.82 83.566) (end 83.82 76.454) (width 0.25) (layer B.Cu) (net 22))
   (segment (start 129.525 92.71) (end 128.27 92.71) (width 0.25) (layer F.Cu) (net 22))
   (segment (start 128.27 91.44) (end 129.54 92.71) (width 0.25) (layer F.Cu) (net 22))
-  (segment (start 83.82 91.44) (end 128.27 91.44) (width 0.25) (layer F.Cu) (net 22))
-  (segment (start 83.82 87.63) (end 83.82 83.566) (width 0.25) (layer B.Cu) (net 22))
-  (segment (start 83.82 91.44) (end 83.82 87.63) (width 0.25) (layer B.Cu) (net 22))
-  (via (at 83.82 91.44) (size 0.8) (drill 0.4) (layers F.Cu B.Cu) (net 22))
+  (segment (start 50.8 91.44) (end 128.27 91.44) (width 0.25) (layer F.Cu) (net 22))
+  (via (at 50.8 91.44) (size 0.8) (drill 0.4) (layers F.Cu B.Cu) (net 22))
+  (segment (start 50.8 91.44) (end 50.8 80.01) (width 0.25) (layer B.Cu) (net 22))
   (segment (start 117.475 92.71) (end 120.65 92.71) (width 0.25) (layer F.Cu) (net 23))
   (segment (start 124.475 92.71) (end 120.65 92.71) (width 0.25) (layer F.Cu) (net 23))
@@
   (segment (start 118.364 88.9) (end 93.726 88.9) (width 0.25) (layer F.Cu) (net 24))
   (segment (start 125.222 88.9) (end 118.364 88.9) (width 0.25) (layer F.Cu) (net 24))
-  (segment (start 92.075 50.8) (end 83.566 50.8) (width 0.25) (layer F.Cu) (net 24))
-  (via (at 92.075 50.8) (size 0.8) (drill 0.4) (layers F.Cu B.Cu) (net 24))
-  (segment (start 92.075 88.9) (end 92.075 50.8) (width 0.25) (layer B.Cu) (net 24))
-  (via (at 92.075 88.9) (size 0.8) (drill 0.4) (layers F.Cu B.Cu) (net 24))
   (segment (start 93.98 88.9) (end 92.075 88.9) (width 0.25) (layer F.Cu) (net 24))
-  (segment (start 93.98 25.4) (end 83.566 25.4) (width 0.25) (layer F.Cu) (net 25))
-  (via (at 93.98 25.4) (size 0.8) (drill 0.4) (layers F.Cu B.Cu) (net 25))
-  (via (at 93.98 86.36) (size 0.8) (drill 0.4) (layers F.Cu B.Cu) (net 25))
-  (segment (start 93.98 86.36) (end 93.98 25.4) (width 0.25) (layer B.Cu) (net 25))
-  (segment (start 118.11 86.36) (end 93.98 86.36) (width 0.25) (layer F.Cu) (net 25))
+  (segment (start 50.8 45.72) (end 50.8 52.07) (width 0.25) (layer B.Cu) (net 24))
+  (segment (start 50.8 52.07) (end 58.42 59.69) (width 0.25) (layer B.Cu) (net 24))
+  (segment (start 59.69 60.96) (end 59.69 88.9) (width 0.25) (layer B.Cu) (net 24))
+  (via (at 59.69 88.9) (size 0.8) (drill 0.4) (layers F.Cu B.Cu) (net 24))
+  (segment (start 58.42 59.69) (end 59.69 60.96) (width 0.25) (layer B.Cu) (net 24))
+  (segment (start 59.69 88.9) (end 92.075 88.9) (width 0.25) (layer F.Cu) (net 24))
   (segment (start 128.27 86.36) (end 118.11 86.36) (width 0.25) (layer F.Cu) (net 25))
   (segment (start 129.54 87.63) (end 128.27 86.36) (width 0.25) (layer F.Cu) (net 25))
+  (segment (start 50.8 12.7) (end 50.8 19.685) (width 0.25) (layer B.Cu) (net 25))
+  (segment (start 50.8 19.685) (end 62.23 31.115) (width 0.25) (layer B.Cu) (net 25))
+  (via (at 62.23 86.36) (size 0.8) (drill 0.4) (layers F.Cu B.Cu) (net 25))
+  (segment (start 62.23 31.115) (end 62.23 86.36) (width 0.25) (layer B.Cu) (net 25))
+  (segment (start 62.23 86.36) (end 99.06 86.36) (width 0.25) (layer F.Cu) (net 25))
+  (segment (start 118.11 86.36) (end 99.06 86.36) (width 0.25) (layer F.Cu) (net 25))
   (segment (start 118.11 87.63) (end 121.92 87.63) (width 0.25) (layer F.Cu) (net 26))
   (segment (start 124.475 87.63) (end 121.92 87.63) (width 0.25) (layer F.Cu) (net 26))
@@
   (via (at 141.224 101.6) (size 0.8) (drill 0.4) (layers F.Cu B.Cu) (net 28))
   (segment (start 143.002 96.52) (end 118.299 96.52) (width 0.25) (layer F.Cu) (net 29))
-  (segment (start 83.82 101.6) (end 83.566 101.854) (width 0.25) (layer F.Cu) (net 29))
-  (segment (start 93.218 96.52) (end 88.138 101.6) (width 0.25) (layer F.Cu) (net 29))
-  (segment (start 88.138 101.6) (end 83.566 101.6) (width 0.25) (layer F.Cu) (net 29))
-  (segment (start 118.364 96.52) (end 93.218 96.52) (width 0.25) (layer F.Cu) (net 29))
+  (segment (start 93.98 96.52) (end 50.8 96.52) (width 0.25) (layer F.Cu) (net 29))
+  (segment (start 118.364 96.52) (end 93.98 96.52) (width 0.25) (layer F.Cu) (net 29))
+  (via (at 50.8 96.52) (size 0.8) (drill 0.4) (layers F.Cu B.Cu) (net 29))
+  (segment (start 93.98 96.52) (end 93.218 96.52) (width 0.25) (layer F.Cu) (net 29))
+  (segment (start 50.8 96.52) (end 50.8 113.792) (width 0.25) (layer B.Cu) (net 29))
   (segment (start 148.017 102.87) (end 152.4 102.87) (width 0.25) (layer F.Cu) (net 30))
-  (segment (start 195.707 50.927) (end 195.834 50.8) (width 0.25) (layer F.Cu) (net 30))
-  (segment (start 152.527 50.8) (end 195.834 50.8) (width 0.25) (layer F.Cu) (net 30))
-  (via (at 152.527 50.8) (size 0.8) (drill 0.4) (layers F.Cu B.Cu) (net 30))
-  (segment (start 152.4 99.06) (end 152.527 50.8) (width 0.25) (layer B.Cu) (net 30))
-  (segment (start 152.4 102.87) (end 152.4 99.06) (width 0.25) (layer B.Cu) (net 30))
+  (segment (start 152.527 45.72) (end 195.834 45.72) (width 0.25) (layer F.Cu) (net 30))
   (via (at 152.4 102.87) (size 0.8) (drill 0.4) (layers F.Cu B.Cu) (net 30))
+  (segment (start 152.4 45.72) (end 152.4 99.06) (width 0.25) (layer B.Cu) (net 30))
+  (segment (start 152.4 99.06) (end 152.4 102.87) (width 0.25) (layer B.Cu) (net 30))
+  (via (at 152.4 45.72) (size 0.8) (drill 0.4) (layers F.Cu B.Cu) (net 30))
   (segment (start 143.067 99.06) (end 142.24 99.06) (width 0.25) (layer F.Cu) (net 31))
   (segment (start 142.24 99.06) (end 120.015 99.06) (width 0.25) (layer F.Cu) (net 31))
-  (via (at 91.44 100.584) (size 0.8) (drill 0.4) (layers F.Cu B.Cu) (net 31))
-  (segment (start 92.964 99.06) (end 91.44 100.584) (width 0.25) (layer F.Cu) (net 31))
   (segment (start 93.472 99.06) (end 92.964 99.06) (width 0.25) (layer F.Cu) (net 31))
-  (segment (start 120.142 99.06) (end 93.472 99.06) (width 0.25) (layer F.Cu) (net 31))
-  (segment (start 83.566 127) (end 91.44 127) (width 0.25) (layer F.Cu) (net 31))
-  (via (at 91.44 127) (size 0.8) (drill 0.4) (layers F.Cu B.Cu) (net 31))
-  (segment (start 91.44 127) (end 91.44 107.95) (width 0.25) (layer B.Cu) (net 31))
-  (segment (start 91.44 107.95) (end 91.44 104.14) (width 0.25) (layer B.Cu) (net 31))
-  (segment (start 91.44 100.584) (end 91.44 104.14) (width 0.25) (layer B.Cu) (net 31))
+  (segment (start 50.8 147.32) (end 50.8 144.145) (width 0.25) (layer B.Cu) (net 31))
+  (segment (start 50.8 144.145) (end 50.8 140.97) (width 0.25) (layer B.Cu) (net 31))
+  (segment (start 50.8 140.97) (end 59.055 132.715) (width 0.25) (layer B.Cu) (net 31))
+  (segment (start 59.055 132.715) (end 59.055 99.06) (width 0.25) (layer B.Cu) (net 31))
+  (via (at 59.055 99.06) (size 0.8) (drill 0.4) (layers F.Cu B.Cu) (net 31))
+  (segment (start 59.055 99.06) (end 95.25 99.06) (width 0.25) (layer F.Cu) (net 31))
+  (segment (start 95.25 99.06) (end 93.472 99.06) (width 0.25) (layer F.Cu) (net 31))
+  (segment (start 120.142 99.06) (end 95.25 99.06) (width 0.25) (layer F.Cu) (net 31))
   (segment (start 170.198 97.79) (end 173.482 97.79) (width 0.25) (layer F.Cu) (net 32))
   (via (at 182.88 97.79) (size 0.8) (drill 0.4) (layers F.Cu B.Cu) (net 32))

Commit message: moving stuff around and working on enclosure
Parts:
- moved C1 11.4 mm to (186.2, 147.3)
- moved J1 11.4 mm to (193.0, 147.3)
- moved J15 3.18 mm to (108.6, 78.1)
Routing:
- net GND: track 38.0 -> 69.9 mm
- net Net-(J5-Pad1): track 132.5 -> 145.2 mm, vias 2 -> 3
- net /P2.7: track 46.4 -> 52.8 mm
- net /P2.6: track 49.3 -> 53.1 mm
- net /P2.5: track 52.3 -> 56.1 mm
- net /P2.0: track 67.2 -> 71.0 mm
- net /P2.4: track 55.2 -> 59.1 mm
- net /P2.3: track 58.2 -> 62.0 mm
- net /P2.1: track 63.9 -> 67.8 mm
- net /P1.6: track 54.4 -> 58.0 mm
- net /P1.4: track 54.5 -> 58.0 mm
- net /P2.2: track 61.0 -> 64.2 mm
- net /P1.7: track 54.0 -> 57.2 mm
- net /P1.5: track 54.3 -> 57.5 mm
