File: board-design/cage-board.sch (KiCad schematic (older format))
At the start: 57 parts, among them J1 Jack-DC, J10 73131-0240, J11 73131-0240, J12 73131-0240, J13 Conn_01x02, J14 Conn_01x02, J15 Conn_02x13_test_points, J16 TB002-500-03BE, J17 TB002-500-03BE, J18 TB002-500-03BE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

Commit message: migrating to branch with new BNC
Parts:
- J10, J11, J12, J4, J5, J6, J8: footprint chen-lab:BNC-Chen -> chen-lab:0731000105 BNC-RightAngle; Item Cost 8.16 -> 1.77; MFN 0731310240 -> 0731000105; Supplier P/N WM5378-ND -> WM5524-ND
Changed lines of the file:
@@
 F 0 "J12" H 5525 3950 50  0000 L CNN
 F 1 "73131-0240" H 5325 4075 50  0000 L CNN
-F 2 "chen-lab:BNC-Chen" H 5425 3950 50  0001 C CNN
-F 3 "https://www.molex.com/pdm_docs/sd/731310240_sd.pdf" H 5425 3950 50  0001 C CNN
+F 2 "chen-lab:0731000105 BNC-RightAngle" H 5425 3950 50  0001 C CNN
+F 3 "https://www.molex.com/pdm_docs/sd/731000105_sd.pdf" H 5425 3950 50  0001 C CNN
 F 4 "Digi-Key" H 5425 3950 50  0001 C CNN "Supplier"
-F 5 "WM5378-ND" H 5425 3950 50  0001 C CNN "Supplier P/N"
-F 6 "0731310240" H 5425 3950 50  0001 C CNN "MFN"
-F 7 "8.16" H 5425 3950 50  0001 C CNN "Item Cost"
+F 5 "WM5524-ND" H 5425 3950 50  0001 C CNN "Supplier P/N"
+F 6 "0731000105" H 5425 3950 50  0001 C CNN "MFN"
+F 7 "1.77" H 5425 3950 50  0001 C CNN "Item Cost"
 	1    5425 3950
 	1    0    0    -1
@@
 F 0 "J6" H 4050 3950 50  0000 L CNN
 F 1 "73131-0240" H 3850 4075 50  0000 L CNN
-F 2 "chen-lab:BNC-Chen" H 3950 3950 50  0001 C CNN
-F 3 "https://www.molex.com/pdm_docs/sd/731310240_sd.pdf" H 3950 3950 50  0001 C CNN
+F 2 "chen-lab:0731000105 BNC-RightAngle" H 3950 3950 50  0001 C CNN
+F 3 "https://www.molex.com/pdm_docs/sd/731000105_sd.pdf" H 3950 3950 50  0001 C CNN
 F 4 "Digi-Key" H 3950 3950 50  0001 C CNN "Supplier"
-F 5 "WM5378-ND" H 3950 3950 50  0001 C CNN "Supplier P/N"
-F 6 "0731310240" H 3950 3950 50  0001 C CNN "MFN"
-F 7 "8.16" H 3950 3950 50  0001 C CNN "Item Cost"
+F 5 "WM5524-ND" H 3950 3950 50  0001 C CNN "Supplier P/N"
+F 6 "0731000105" H 3950 3950 50  0001 C CNN "MFN"
+F 7 "1.77" H 3950 3950 50  0001 C CNN "Item Cost"
 	1    3950 3950
 	1    0    0    -1
@@
 F 0 "J5" H 4125 7075 50  0000 L CNN
 F 1 "73131-0240" H 3925 7200 50  0000 L CNN
-F 2 "chen-lab:BNC-Chen" H 4025 7075 50  0001 C CNN
-F 3 "https://www.molex.com/pdm_docs/sd/731310240_sd.pdf" H 4025 7075 50  0001 C CNN
+F 2 "chen-lab:0731000105 BNC-RightAngle" H 4025 7075 50  0001 C CNN
+F 3 "https://www.molex.com/pdm_docs/sd/731000105_sd.pdf" H 4025 7075 50  0001 C CNN
 F 4 "Digi-Key" H 4025 7075 50  0001 C CNN "Supplier"
-F 5 "WM5378-ND" H 4025 7075 50  0001 C CNN "Supplier P/N"
-F 6 "0731310240" H 4025 7075 50  0001 C CNN "MFN"
-F 7 "8.16" H 4025 7075 50  0001 C CNN "Item Cost"
+F 5 "WM5524-ND" H 4025 7075 50  0001 C CNN "Supplier P/N"
+F 6 "0731000105" H 4025 7075 50  0001 C CNN "MFN"
+F 7 "1.77" H 4025 7075 50  0001 C CNN "Item Cost"
 	1    4025 7075
 	1    0    0    -1
@@
 F 0 "J11" H 6100 7025 50  0000 L CNN
 F 1 "73131-0240" H 5900 7150 50  0000 L CNN
-F 2 "chen-lab:BNC-Chen" H 6000 7025 50  0001 C CNN
-F 3 "https://www.molex.com/pdm_docs/sd/731310240_sd.pdf" H 6000 7025 50  0001 C CNN
+F 2 "chen-lab:0731000105 BNC-RightAngle" H 6000 7025 50  0001 C CNN
+F 3 "https://www.molex.com/pdm_docs/sd/731000105_sd.pdf" H 6000 7025 50  0001 C CNN
 F 4 "Digi-Key" H 6000 7025 50  0001 C CNN "Supplier"
-F 5 "WM5378-ND" H 6000 7025 50  0001 C CNN "Supplier P/N"
-F 6 "0731310240" H 6000 7025 50  0001 C CNN "MFN"
-F 7 "8.16" H 6000 7025 50  0001 C CNN "Item Cost"
+F 5 "WM5524-ND" H 6000 7025 50  0001 C CNN "Supplier P/N"
+F 6 "0731000105" H 6000 7025 50  0001 C CNN "MFN"
+F 7 "1.77" H 6000 7025 50  0001 C CNN "Item Cost"
 	1    6000 7025
 	1    0    0    -1
@@
 F 0 "J4" H 3375 4975 50  0000 L CNN
 F 1 "73131-0240" H 3175 5100 50  0000 L CNN
-F 2 "chen-lab:BNC-Chen" H 3275 4975 50  0001 C CNN
-F 3 "https://www.molex.com/pdm_docs/sd/731310240_sd.pdf" H 3275 4975 50  0001 C CNN
+F 2 "chen-lab:0731000105 BNC-RightAngle" H 3275 4975 50  0001 C CNN
+F 3 "https://www.molex.com/pdm_docs/sd/731000105_sd.pdf" H 3275 4975 50  0001 C CNN
 F 4 "Digi-Key" H 3275 4975 50  0001 C CNN "Supplier"
-F 5 "WM5378-ND" H 3275 4975 50  0001 C CNN "Supplier P/N"
-F 6 "0731310240" H 3275 4975 50  0001 C CNN "MFN"
-F 7 "8.16" H 3275 4975 50  0001 C CNN "Item Cost"
+F 5 "WM5524-ND" H 3275 4975 50  0001 C CNN "Supplier P/N"
+F 6 "0731000105" H 3275 4975 50  0001 C CNN "MFN"
+F 7 "1.77" H 3275 4975 50  0001 C CNN "Item Cost"
 	1    3275 4975
 	1    0    0    -1
@@
 F 0 "J8" H 4250 5000 50  0000 L CNN
 F 1 "73131-0240" H 4050 5125 50  0000 L CNN
-F 2 "chen-lab:BNC-Chen" H 4150 5000 50  0001 C CNN
-F 3 "https://www.molex.com/pdm_docs/sd/731310240_sd.pdf" H 4150 5000 50  0001 C CNN
+F 2 "chen-lab:0731000105 BNC-RightAngle" H 4150 5000 50  0001 C CNN
+F 3 "https://www.molex.com/pdm_docs/sd/731000105_sd.pdf" H 4150 5000 50  0001 C CNN
 F 4 "Digi-Key" H 4150 5000 50  0001 C CNN "Supplier"
-F 5 "WM5378-ND" H 4150 5000 50  0001 C CNN "Supplier P/N"
-F 6 "0731310240" H 4150 5000 50  0001 C CNN "MFN"
-F 7 "8.16" H 4150 5000 50  0001 C CNN "Item Cost"
+F 5 "WM5524-ND" H 4150 5000 50  0001 C CNN "Supplier P/N"
+F 6 "0731000105" H 4150 5000 50  0001 C CNN "MFN"
+F 7 "1.77" H 4150 5000 50  0001 C CNN "Item Cost"
 	1    4150 5000
 	1    0    0    -1
@@
 F 0 "J10" H 5175 5000 50  0000 L CNN
 F 1 "73131-0240" H 4975 5125 50  0000 L CNN
-F 2 "chen-lab:BNC-Chen" H 5075 5000 50  0001 C CNN
-F 3 "https://www.molex.com/pdm_docs/sd/731310240_sd.pdf" H 5075 5000 50  0001 C CNN
+F 2 "chen-lab:0731000105 BNC-RightAngle" H 5075 5000 50  0001 C CNN
+F 3 "https://www.molex.com/pdm_docs/sd/731000105_sd.pdf" H 5075 5000 50  0001 C CNN
 F 4 "Digi-Key" H 5075 5000 50  0001 C CNN "Supplier"
-F 5 "WM5378-ND" H 5075 5000 50  0001 C CNN "Supplier P/N"
-F 6 "0731310240" H 5075 5000 50  0001 C CNN "MFN"
-F 7 "8.16" H 5075 5000 50  0001 C CNN "Item Cost"
+F 5 "WM5524-ND" H 5075 5000 50  0001 C CNN "Supplier P/N"
+F 6 "0731000105" H 5075 5000 50  0001 C CNN "MFN"
+F 7 "1.77" H 5075 5000 50  0001 C CNN "Item Cost"
 	1    5075 5000
 	1    0    0    -1
